File: pcb/AnitaHuang.kicad_pcb (KiCad board)
At the start: 2 copper layers, 65 x 56 mm, 11 parts, among them J1 HBRIDGE_LEFT, J2 HBRIDGE_RIGHT, J3 MOTOR_A, J4 MOTOR_B, J5 SERVO_1, J6 SERVO_2, P1 Conn_02x20_Odd_Even

Commit message: Autonomous push
Routing:
- net +5V: track 112.8 -> 90.7 mm
Changed lines of the file:
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@@
 	)
 	(segment
-		(start 108.85 73.65)
-		(end 99.79 64.59)
+		(start 85.74 76.1)
+		(end 85.9 76.1)
 		(width 0.2)
 		(layer "F.Cu")
@@
 	)
 	(segment
-		(start 82.64 49.24)
-		(end 80.1 49.24)
-		(width 0.2)
-		(layer "F.Cu")
-		(net 2)
-	)
-	(segment
-		(start 85.74 76.1)
-		(end 85.9 76.1)
+		(start 90.73 73.65)
+		(end 108.85 73.65)
 		(width 0.2)
 		(layer "F.Cu")
@@
 	)
 	(segment
-		(start 80.1 49.24)
-		(end 81.74 47.6)
+		(start 82.64 49.24)
+		(end 82.76 49.24)
 		(width 0.2)
 		(layer "F.Cu")
@@
 	)
 	(segment
-		(start 99.79 64.59)
-		(end 88.28 76.1)
+		(start 80.1 49.24)
+		(end 82.64 49.24)
 		(width 0.2)
 		(layer "F.Cu")
@@
 	)
 	(segment
-		(start 102.946346 47.6)
-		(end 104.11 48.763654)
+		(start 88.28 76.1)
+		(end 90.73 73.65)
 		(width 0.2)
 		(layer "F.Cu")
@@
 	)
 	(segment
-		(start 99.79 60.623654)
-		(end 99.79 64.59)
+		(start 84.03 50.63)
+		(end 84.03 74.39)
 		(width 0.2)
 		(layer "F.Cu")
@@
 	)
 	(segment
-		(start 81.74 47.6)
-		(end 102.946346 47.6)
+		(start 84.03 74.39)
+		(end 85.74 76.1)
 		(width 0.2)
 		(layer "F.Cu")
@@
 	)
 	(segment
-		(start 104.11 56.303654)
-		(end 99.79 60.623654)
+		(start 82.64 49.24)
+		(end 84.03 50.63)
 		(width 0.2)
 		(layer "F.Cu")
@@
 		(width 0.2)
 		(layer "F.Cu")
-		(net 2)
-	)
-	(segment
-		(start 104.11 48.763654)
-		(end 104.11 56.303654)
-		(width 0.2)
-		(layer "F.Cu")
