File: pcb/Lec18-PCB_kicad.kicad_sch (KiCad schematic)
At the start: 5 parts, among them P1 Conn_02x20_Odd_Even

Commit message: Fork Lift
Parts:
- added J1: HBRIDGE_LEFT, Connector_PinSocket_2.54mm:PinSocket_1x08_P2.54mm_Vertical, symbol Connector_Generic:Conn_01x08
- added J2: HBRIDGE_RIGHT, Connector_PinSocket_2.54mm:PinSocket_1x08_P2.54mm_Vertical, symbol Connector_Generic:Conn_01x08
- added J3: MOTOR_A, Connector_PinHeader_2.54mm:PinHeader_1x02_P2.54mm_Vertical, symbol Connector_Generic:Conn_01x02
- added J4: MOTOR_B, Connector_PinHeader_2.54mm:PinHeader_1x02_P2.54mm_Vertical, symbol Connector_Generic:Conn_01x02
- added J5: SERVO_1, Connector_PinHeader_2.54mm:PinHeader_1x03_P2.54mm_Vertical, symbol Connector_Generic:Conn_01x03
- added J6: SERVO_2, Connector_PinHeader_2.54mm:PinHeader_1x03_P2.54mm_Vertical, symbol Connector_Generic:Conn_01x03
Connections:
- net +5V: now also J1.1 (Pin_1), J1.2 (Pin_2), J5.2 (Pin_2), J6.2 (Pin_2)
- net GND: now also J1.3 (Pin_3), J1.8 (Pin_8), J2.8 (Pin_8), J5.1 (Pin_1), J6.1 (Pin_1)
- net GPIO12(PWM0): now also J2.7 (Pin_7)
- net GPIO13(PWM1): now also J5.3 (Pin_3)
- net GPIO18(GEN1)(PWM0): now also J2.1 (Pin_1)
- net GPIO19(SPI1_MISO): now also J6.3 (Pin_3)
- net GPIO24(GEN5): now also J2.4 (Pin_4)
- net GPIO17(GEN0) renamed AI1
- net AI1: now also J2.3 (Pin_3)
- net GPIO22(GEN3) renamed BI1
- net BI1: now also J2.5 (Pin_5)
- net GPIO23(GEN4) renamed BI2
- net BI2: now also J2.6 (Pin_6)
- net GPIO27(GEN2) renamed AI2
- net AI2: now also J2.2 (Pin_2)
- new net A01: J1.4 (Pin_4), J3.1 (Pin_1)
- new net A02: J1.5 (Pin_5), J3.2 (Pin_2)
- new net B01: J1.7 (Pin_7), J4.1 (Pin_1)
- new net B02: J1.6 (Pin_6), J4.2 (Pin_2)

Commit message: Autonomous push
Connections:
- net +5V: no longer J1.1 (Pin_1)
- new net VM: J1.1 (Pin_1)
Changed lines of the file:
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@@
-		)
-	)
-	(label "VM"
-		(at 93.98 27.94 0)
-		(fields_autoplaced yes)
-		(effects
-			(font
-				(size 1.27 1.27)
-			)
-			(justify left bottom)
 		)
 	)
